File: BrookHitbox/BrookHitbox.kicad_pcb (KiCad board)
At the start: 2 copper layers, 24 parts

Commit message: mounting hole placement
Parts:
- moved H3 321.0 mm to (378.5, 223.5)
- moved H4 271.9 mm to (378.5, 71.1)
- moved H1 173.0 mm to (50.8, 223.5)
- moved H7 140.7 mm to (218.4, 164.2)
- moved H5 126.8 mm to (181.4, 164.2)
- moved H8 88.3 mm to (218.4, 76.2)
- moved H6 66.3 mm to (181.4, 76.2)
- moved BrookConnection1 46.1 mm to (248.9, 118.0)
- moved H2 44.7 mm to (50.8, 71.1)
- moved SW_L2 9.89 mm to (363.4, 128.6)
- moved SW_PSXBOX1 9.89 mm to (252.6, 204.8)
- moved SW_SELECT1 9.89 mm to (252.6, 173.7)
- moved SW_L1 9.89 mm to (363.4, 101.0)
- moved SW_SQUARE1 9.89 mm to (282.3, 93.9)
- moved SW_X1 9.89 mm to (282.3, 121.5)
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Changed lines of the file:
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@@
   (net 16 "GND")
   (footprint "MountingHole:MountingHole_2.2mm_M2" (layer "F.Cu")
-    (at 93.2719 55.8024)
+    (at 50.8 223.52)
     (descr "Mounting Hole 2.2mm, no annular, M2")
     (tags "mounting hole 2.2mm no annular m2")
@@
   )
   (footprint "Button_Switch_Keyboard:SW_Cherry_MX_1.00u_PCB" (layer "F.Cu")
-    (at 306.608 72.295)
+    (at 308.78 81.941)
     (descr "Cherry MX keyswitch, 1.00u, PCB mount, http://cherryamericas.com/wp-content/uploads/2014/12/mx_cat.pdf")
     (tags "Cherry MX keyswitch 1.00u PCB")
@@
   )
   (footprint "Button_Switch_Keyboard:SW_Cherry_MX_1.00u_PCB" (layer "F.Cu")
-    (at 250.388 195.195)
+    (at 252.56 204.841)
     (descr "Cherry MX keyswitch, 1.00u, PCB mount, http://cherryamericas.com/wp-content/uploads/2014/12/mx_cat.pdf")
     (tags "Cherry MX keyswitch 1.00u PCB")
@@
   )
   (footprint "Button_Switch_Keyboard:SW_Cherry_MX_1.00u_PCB" (layer "F.Cu")
-    (at 250.388 164.01)
+    (at 252.56 173.656)
     (descr "Cherry MX keyswitch, 1.00u, PCB mount, http://cherryamericas.com/wp-content/uploads/2014/12/mx_cat.pdf")
     (tags "Cherry MX keyswitch 1.00u PCB")
@@
   )
   (footprint "Button_Switch_Keyboard:SW_Cherry_MX_1.00u_PCB" (layer "F.Cu")
-    (at 280.09 84.291)
+    (at 282.262 93.937)
     (descr "Cherry MX keyswitch, 1.00u, PCB mount, http://cherryamericas.com/wp-content/uploads/2014/12/mx_cat.pdf")
     (tags "Cherry MX keyswitch 1.00u PCB")
@@
   )
   (footprint "MountingHole:MountingHole_2.2mm_M2" (layer "F.Cu")
-    (at 95.5319 70.6024)
+    (at 50.8 71.12)
     (descr "Mounting Hole 2.2mm, no annular, M2")
     (tags "mounting hole 2.2mm no annular m2")
@@
   )
   (footprint "Button_Switch_Keyboard:SW_Cherry_MX_1.00u_PCB" (layer "F.Cu")
-    (at 334.963 75.27)
+    (at 337.135 84.916)
     (descr "Cherry MX keyswitch, 1.00u, PCB mount, http://cherryamericas.com/wp-content/uploads/2014/12/mx_cat.pdf")
     (tags "Cherry MX keyswitch 1.00u PCB")
@@
   )
   (footprint "MountingHole:MountingHole_2.2mm_M2" (layer "F.Cu")
-    (at 130.3119 71.2524)
+    (at 218.44 76.2)
     (descr "Mounting Hole 2.2mm, no annular, M2")
     (tags "mounting hole 2.2mm no annular m2")
@@
   )
   (footprint "Button_Switch_Keyboard:SW_Cherry_MX_1.00u_PCB" (layer "F.Cu")
-    (at 306.608 99.905)
+    (at 308.78 109.551)
     (descr "Cherry MX keyswitch, 1.00u, PCB mount, http://cherryamericas.com/wp-content/uploads/2014/12/mx_cat.pdf")
     (tags "Cherry MX keyswitch 1.00u PCB")
@@
   )
   (footprint "Button_Switch_Keyboard:SW_Cherry_MX_1.00u_PCB" (layer "F.Cu")
-    (at 94.724 100.511)
+    (at 96.896 110.157)
     (descr "Cherry MX keyswitch, 1.00u, PCB mount, http://cherryamericas.com/wp-content/uploads/2014/12/mx_cat.pdf")
     (tags "Cherry MX keyswitch 1.00u PCB")
@@
   )
   (footprint "MountingHole:MountingHole_2.2mm_M2" (layer "F.Cu")
-    (at 127.8219 56.5624)
+    (at 218.44 164.2)
     (descr "Mounting Hole 2.2mm, no annular, M2")
     (tags "mounting hole 2.2mm no annular m2")
@@
   )
   (footprint "Button_Switch_Keyboard:SW_Cherry_MX_1.00u_PCB" (layer "F.Cu")
-    (at 361.186 118.916)
+    (at 363.358 128.562)
     (descr "Cherry MX keyswitch, 1.00u, PCB mount, http://cherryamericas.com/wp-content/uploads/2014/12/mx_cat.pdf")
     (tags "Cherry MX keyswitch 1.00u PCB")
@@
   )
   (footprint "Button_Switch_Keyboard:SW_Cherry_MX_1.00u_PCB" (layer "F.Cu")
-    (at 121.296 112.274)
+    (at 123.468 121.92)
     (descr "Cherry MX keyswitch, 1.00u, PCB mount, http://cherryamericas.com/wp-content/uploads/2014/12/mx_cat.pdf")
     (tags "Cherry MX keyswitch 1.00u PCB")
@@
   )
   (footprint "Button_Switch_Keyboard:SW_Cherry_MX_1.00u_PCB" (layer "F.Cu")
-    (at 66.368 103.237)
+    (at 68.54 112.883)
     (descr "Cherry MX keyswitch, 1.00u, PCB mount, http://cherryamericas.com/wp-content/uploads/2014/12/mx_cat.pdf")
     (tags "Cherry MX keyswitch 1.00u PCB")
@@
   )
   (footprint "Button_Switch_Keyboard:SW_Cherry_MX_1.00u_PCB" (layer "F.Cu")
-    (at 201.028 112.274)
+    (at 203.2 121.92)
     (descr "Cherry MX keyswitch, 1.00u, PCB mount, http://cherryamericas.com/wp-content/uploads/2014/12/mx_cat.pdf")
     (tags "Cherry MX keyswitch 1.00u PCB")
@@
   )
   (footprint "MountingHole:MountingHole_2.2mm_M2" (layer "F.Cu")
-    (at 115.1619 73.1724)
+    (at 181.44 76.2)
     (descr "Mounting Hole 2.2mm, no annular, M2")
     (tags "mounting hole 2.2mm no annular m2")
@@
   )
   (footprint "Button_Switch_Keyboard:SW_Cherry_MX_1.00u_PCB" (layer "F.Cu")
-    (at 334.963 102.88)
+    (at 337.135 112.526)
     (descr "Cherry MX keyswitch, 1.00u, PCB mount, http://cherryamericas.com/wp-content/uploads/2014/12/mx_cat.pdf")
     (tags "Cherry MX keyswitch 1.00u PCB")
@@
   )
   (footprint "Button_Switch_Keyboard:SW_Cherry_MX_1.00u_PCB" (layer "F.Cu")
-    (at 280.09 111.9)
+    (at 282.262 121.546)
     (descr "Cherry MX keyswitch, 1.00u, PCB mount, http://cherryamericas.com/wp-content/uploads/2014/12/mx_cat.pdf")
     (tags "Cherry MX keyswitch 1.00u PCB")
@@
   )
   (footprint "MountingHole:MountingHole_2.2mm_M2" (layer "F.Cu")
-    (at 106.5819 73.9024)
+    (at 378.46 71.12)
     (descr "Mounting Hole 2.2mm, no annular, M2")
     (tags "mounting hole 2.2mm no annular m2")
@@
   )
   (footprint "BrookHitboxFootprints:BrookConn16" (layer "F.Cu")
-    (at 219.8619 82.2224 -90)
+    (at 248.92 118.05 -90)
     (property "Sheetfile" "BrookHitbox.kicad_sch")
     (property "Sheetname" "")
@@
   )
   (footprint "MountingHole:MountingHole_2.2mm_M2" (layer "F.Cu")
-    (at 104.7319 55.9124)
+    (at 378.46 223.52)
     (descr "Mounting Hole 2.2mm, no annular, M2")
     (tags "mounting hole 2.2mm no annular m2")
@@
   )
   (footprint "MountingHole:MountingHole_2.2mm_M2" (layer "F.Cu")
-    (at 114.0119 56.8324)
+    (at 181.44 164.2)
     (descr "Mounting Hole 2.2mm, no annular, M2")
     (tags "mounting hole 2.2mm no annular m2")
@@
   )
   (footprint "Button_Switch_Keyboard:SW_Cherry_MX_1.00u_PCB" (layer "F.Cu")
-    (at 361.186 91.306)
+    (at 363.358 100.952)
     (descr "Cherry MX keyswitch, 1.00u, PCB mount, http://cherryamericas.com/wp-content/uploads/2014/12/mx_cat.pdf")
     (tags "Cherry MX keyswitch 1.00u PCB")
@@
   )
   (footprint "Button_Switch_Keyboard:SW_Cherry_MX_1.00u_PCB" (layer "F.Cu")
-    (at 128.255 179.425)
-    (descr "Cherry MX keyswitch, 1.00u, PCB mount, http://cherryamericas.com/wp-content/uploads/2014/12/mx_cat.pdf")
-    (tags "Cherry MX keyswitch 1.00u PCB")
+    (at 130.427 189.071)
+    (descr "Cherry MX keyswitch, 1.00u, PCB mount, http://cherryamericas.com/wp-content/uploads/2014/12/mx_cat.pdf")
+    (tags "Cherry MX keyswitch 1.00u PCB")

Commit message: edge cuts
Parts:
- moved H4 0.25 mm to (378.2, 71.2)
- moved H3 0.21 mm to (378.2, 223.5)
- moved H2 0.14 mm to (50.8, 71.2)
- moved H1 0.05 mm to (50.8, 223.5)
Other:
- board outline added: 333.5 x 158.2 mm
Changed lines of the file:
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@@
   (net 16 "GND")
   (footprint "MountingHole:MountingHole_2.2mm_M2" (layer "F.Cu")
-    (at 50.8 223.52)
+    (at 50.75 223.5)
     (descr "Mounting Hole 2.2mm, no annular, M2")
     (tags "mounting hole 2.2mm no annular m2")
@@
   )
   (footprint "MountingHole:MountingHole_2.2mm_M2" (layer "F.Cu")
-    (at 50.8 71.12)
+    (at 50.75 71.25)
     (descr "Mounting Hole 2.2mm, no annular, M2")
     (tags "mounting hole 2.2mm no annular m2")
@@
   )
   (footprint "MountingHole:MountingHole_2.2mm_M2" (layer "F.Cu")
-    (at 378.46 71.12)
+    (at 378.25 71.25)
     (descr "Mounting Hole 2.2mm, no annular, M2")
     (tags "mounting hole 2.2mm no annular m2")
@@
   )
   (footprint "MountingHole:MountingHole_2.2mm_M2" (layer "F.Cu")
-    (at 378.46 223.52)
+    (at 378.25 223.5)
     (descr "Mounting Hole 2.2mm, no annular, M2")
     (tags "mounting hole 2.2mm no annular m2")
@@
     )
   )
+  (gr_arc (start 381.25 223.5) (mid 380.37132 225.62132) (end 378.25 226.5)
+    (stroke (width 0.1) (type default)) (layer "Edge.Cuts"))
+  (gr_line (start 378.25 68.25) (end 50.75 68.25)
+    (stroke (width 0.1) (type default)) (layer "Edge.Cuts"))
+  (gr_line (start 378.25 226.5) (end 50.75 226.5)
+    (stroke (width 0.1) (type default)) (layer "Edge.Cuts"))
+  (gr_line (start 381.25 71.25) (end 381.25 223.5)
+    (stroke (width 0.1) (type default)) (layer "Edge.Cuts"))
+  (gr_arc (start 378.25 68.25) (mid 380.37132 69.12868) (end 381.25 71.25)
+    (stroke (width 0.1) (type default)) (layer "Edge.Cuts"))
+  (gr_arc (start 47.75 71.25) (mid 48.62868 69.12868) (end 50.75 68.25)
+    (stroke (width 0.1) (type default)) (layer "Edge.Cuts"))
+  (gr_arc (start 50.75 226.5) (mid 48.62868 225.62132) (end 47.75 223.5)
+    (stroke (width 0.1) (type default)) (layer "Edge.Cuts"))
+  (gr_line (start 47.75 71.25) (end 47.75 223.5)
+    (stroke (width 0.1) (type default)) (layer "Edge.Cuts"))
 )

Commit message: traces
Parts:
- BrookConnection1: moved to B.Cu
Routing:
- net GND: track 0.00 -> 601.4 mm, vias 0 -> 1
- net /LFT: track 0.00 -> 185.4 mm, vias 0 -> 2
- net /UP: track 0.00 -> 160.0 mm, vias 0 -> 2
- net /DWN: track 0.00 -> 153.4 mm
- net /L1: track 0.00 -> 152.8 mm, vias 0 -> 2
- net /RT: track 0.00 -> 129.9 mm
- net /L2: track 0.00 -> 118.2 mm
- net /R1: track 0.00 -> 113.3 mm, vias 0 -> 2
- net /R2: track 0.00 -> 108.0 mm, vias 0 -> 4
- net /PS: track 0.00 -> 105.7 mm, vias 0 -> 2
- net /TRI: track 0.00 -> 78.5 mm, vias 0 -> 2
- net /SEL: track 0.00 -> 69.5 mm, vias 0 -> 2
- net /CIR: track 0.00 -> 66.2 mm, vias 0 -> 2
- net /STA: track 0.00 -> 48.3 mm
- net /SQU: track 0.00 -> 43.0 mm
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
Commit message: generated gerber
Parts:
- moved H6 4.98 mm to (182.0, 71.2)
- moved H5 4.98 mm to (182.0, 159.2)
- moved H7 4.98 mm to (219.0, 159.2)
- moved H8 4.73 mm to (219.0, 71.5)
Other:
- board text added: "VL-UFB"
Changed lines of the file:
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@@
       (usegerberattributes true)
       (usegerberadvancedattributes true)
-      (creategerberjobfile true)
+      (creategerberjobfile false)
       (dashed_line_dash_ratio 12.000000)
       (dashed_line_gap_ratio 3.000000)
@@
       (outputformat 1)
       (mirror false)
-      (drillshape 1)
+      (drillshape 0)
       (scaleselection 1)
-      (outputdirectory "")
+      (outputdirectory "../manufacturing/")
     )
   )
@@
   )
   (footprint "MountingHole:MountingHole_2.2mm_M2" (layer "F.Cu")
-    (at 218.44 76.2)
+    (at 219 71.5)
     (descr "Mounting Hole 2.2mm, no annular, M2")
     (tags "mounting hole 2.2mm no annular m2")
@@
   )
   (footprint "MountingHole:MountingHole_2.2mm_M2" (layer "F.Cu")
-    (at 218.44 164.2)
+    (at 219 159.25)
     (descr "Mounting Hole 2.2mm, no annular, M2")
     (tags "mounting hole 2.2mm no annular m2")
@@
   )
   (footprint "MountingHole:MountingHole_2.2mm_M2" (layer "F.Cu")
-    (at 181.44 76.2)
+    (at 182 71.25)
     (descr "Mounting Hole 2.2mm, no annular, M2")
     (tags "mounting hole 2.2mm no annular m2")
@@
   )
   (footprint "MountingHole:MountingHole_2.2mm_M2" (layer "F.Cu")
-    (at 181.44 164.2)
+    (at 182 159.25)
     (descr "Mounting Hole 2.2mm, no annular, M2")
     (tags "mounting hole 2.2mm no annular m2")
@@
     (property "Sheetname" "")
     (attr through_hole)
-    (fp_text reference "SW_UP1" (at -2.54 -2.54) (layer "F.SilkS")
-        (effects (font (size 1 1) (thickness 0.15)))
-    )
-    (fp_text value "~" (at -2.54 12.954) (layer "F.Fab") hide
-        (effects (font (size 1 1) (thickness 0.15)))
-    )
-    (fp_text user "${REFERENCE}" (at -2.54 -2.54) (layer "F.Fab")
+    (fp_text reference "SW_UP1" (at -2.427 -2.821) (layer "F.SilkS")
+        (effects (font (size 1 1) (thickness 0.15)))
+    )
+    (fp_text value "~" (at -2.54 12.954) (layer "F.Fab") hide
+        (effects (font (size 1 1) (thickness 0.15)))
+    )
+    (fp_text user "${REFERENCE}" (at -2.427 -2.821) (layer "F.Fab")
         (effects (font (size 1 1) (thickness 0.15)))
     )
@@
   (gr_line (start 47.75 71.25) (end 47.75 223.5)
     (stroke (width 0.1) (type default)) (layer "Edge.Cuts"))
+  (gr_text "VL-UFB" (at 72.75 221.25) (layer "F.SilkS")
+    (effects (font (size 5 5) (thickness 0.15)) (justify left bottom))
+  )
   (segment (start 100.253 106.8) (end 96.896 110.157) (width 0.3) (layer "B.Cu") (net 1))
   (segment (start 248.92 106.8) (end 100.253 106.8) (width 0.3) (layer "B.Cu") (net 1))
@@
   (segment (start 302.43 84.481) (end 302.43 112.091) (width 0.3) (layer "F.Cu") (net 16))
   (segment (start 87.322233 115.423) (end 90.048233 112.697) (width 0.3) (layer "F.Cu") (net 16))
+  (segment (start 337.75 103.492) (end 334.293 103.492) (width 0.3) (layer "F.Cu") (net 16))
   (segment (start 108 132.022366) (end 115.562366 124.46) (width 0.3) (layer "F.Cu") (net 16))
   (segment (start 90.546 112.697) (end 105.355 112.697) (width 0.3) (layer "F.Cu") (net 16))
@@
   (segment (start 330.785 87.456) (end 327.81 84.481) (width 0.3) (layer "F.Cu") (net 16))
   (segment (start 235.5 129.25) (end 230.71 124.46) (width 0.3) (layer "F.Cu") (net 16))
-  (segment (start 357.008 103.492) (end 334.293 103.492) (width 0.3) (layer "F.Cu") (net 16))
   (segment (start 264.664 124.086) (end 257.54 131.21) (width 0.3) (layer "F.Cu") (net 16))
   (segment (start 62.19 115.423) (end 87.322233 115.423) (width 0.3) (layer "F.Cu") (net 16))
@@
   (segment (start 334.293 103.492) (end 330.785 107) (width 0.3) (layer "F.Cu") (net 16))
   (segment (start 246.21 207.381) (end 246.21 176.196) (width 0.3) (layer "F.Cu") (net 16))
+  (segment (start 357.008 103.492) (end 337.75 103.492) (width 0.3) (layer "F.Cu") (net 16))
   (segment (start 124.077 191.611) (end 191.228 124.46) (width 0.3) (layer "F.Cu") (net 16))
   (via (at 244.25 129.25) (size 0.7) (drill 0.3) (layers "F.Cu" "B.Cu") (net 16))
